File: sp3485-breakout.sch (KiCad schematic (older format))
At the start: 5 parts, among them J1 Conn_01x04, J2 Conn_01x04, U1 SP3485CN

Commit message: Add condensor
Parts:
- added C1: 0.1u, Capacitor_SMD:C_0402_1005Metric, symbol Device:C
- R1: footprint Resistor_SMD:R_0603_1608Metric -> Resistor_SMD:R_0402_1005Metric
Connections:
- net GND: now also C1.2
- net VCC: now also C1.1
Changed lines of the file:
@@
 F 0 "R1" H 6870 3346 50  0000 L CNN
 F 1 "220" H 6870 3255 50  0000 L CNN
-F 2 "Resistor_SMD:R_0603_1608Metric" V 6730 3300 50  0001 C CNN
+F 2 "Resistor_SMD:R_0402_1005Metric" V 6730 3300 50  0001 C CNN
 F 3 "~" H 6800 3300 50  0001 C CNN
 	1    6800 3300
@@
 Wire Wire Line
 	6800 2850 7200 2850
+$Comp
+L Device:C C1
+U 1 1 61DF0853
+P 7550 2450
+F 0 "C1" H 7665 2496 50  0000 L CNN
+F 1 "0.1u" H 7665 2405 50  0000 L CNN
+F 2 "Capacitor_SMD:C_0402_1005Metric" H 7588 2300 50  0001 C CNN
+F 3 "~" H 7550 2450 50  0001 C CNN
+	1    7550 2450
+	1    0    0    -1
+$EndComp
+$Comp
+L power:GND #PWR0104
+U 1 1 61DF0A11
+P 7550 2600
+F 0 "#PWR0104" H 7550 2350 50  0001 C CNN
+F 1 "GND" H 7555 2427 50  0000 C CNN
+F 2 "" H 7550 2600 50  0001 C CNN
+F 3 "" H 7550 2600 50  0001 C CNN
+	1    7550 2600
+	1    0    0    -1
+$EndComp
+$Comp
+L power:VCC #PWR0105
+U 1 1 61DF0D23
+P 7550 2300
+F 0 "#PWR0105" H 7550 2150 50  0001 C CNN
+F 1 "VCC" H 7565 2473 50  0000 C CNN
+F 2 "" H 7550 2300 50  0001 C CNN
+F 3 "" H 7550 2300 50  0001 C CNN
+	1    7550 2300
+	1    0    0    -1
+$EndComp
 $EndSCHEMATC
